Commit message: modified world file to include sensor plugin, added mission.py file to implement the requested behaviour, for now only search phase is working

File: urdf/mogi_bot.urdf (robot description, URDF)
Before this commit: robot mogi_bot, 9 links, 8 joints
Links:
- link base_link: geometry collision box size=.4 .2 .1; collision sphere radius=0.0499
- link left_wheel: geometry collision cylinder length=.05 radius=.1; visual mesh filename=package://erl_assignment_1/meshes/wheel.dae
- link right_wheel: geometry collision cylinder length=.05 radius=.1; visual mesh filename=package://erl_assignment_1/meshes/wheel.dae
- link scan_link: geometry collision box size=0.1 0.1 0.1; visual mesh filename=package://erl_assignment_1/meshes/lidar.dae

Commit message: added short mission file in which robt does not get closer to the markers, added launch files for every combination of mission, modified urdf to set correct lidar position, modified mission node to open a window with the modified images, rotation speed changed at 0.4

File: urdf/mogi_bot.urdf (robot description, URDF)
Before this commit: robot mogi_bot, 9 links, 8 joints
Joints:
- joint scan_joint: origin (none) -> xyz=0 0 0.12 rpy=0 0 0
